Commit message: initial commit for mm changes

File: wamv_description/urdf/wamv_base.urdf.xacro (robot description, xacro)
@@ -91,12 +91,18 @@
     <visual>
       <geometry>
-        <mesh filename="package://wamv_description/models/WAM-V-Base/mesh/WAM-V-Base.dae"/>
+        <mesh filename="package://wamv_description/models/hovercraft/model.dae"/>
       </geometry>
     </visual>
+	<collision>
+		<geometry>
+			<mesh filename="package://wamv_description/models/hovercraft/model.dae"/>
+		</geometry>
+	</collision>
     <!-- Left base collisions -->
-    <xacro:main_collisions prefix="left" reflect="1" />
+    <!--><xacro:main_collisions prefix="left" reflect="1" /><-->
     <!-- Right side collisions -->
-    <xacro:main_collisions prefix="right" reflect="-1" />
+    <!--><xacro:main_collisions prefix="right" reflect="-1" /><-->
      <!-- Top base -->
+<!-->
     <collision name="top_base">
       <origin xyz="0 -0 1.25" rpy="0 0 0" />
@@ -105,4 +111,5 @@
       </geometry>
     </collision>
+<-->
     <inertial>
       <!-- From WAM-V spec sheet -->

File: wamv_gazebo/urdf/macros.xacro (robot description, xacro)
@@ -13,4 +13,3 @@
   <xacro:include filename="$(find wamv_gazebo)/urdf/sensors/lidar.xacro" />
   <xacro:include filename="$(find wamv_gazebo)/urdf/sensors/wamv_p3d.xacro" />
-  <xacro:include filename="$(find wamv_gazebo)/urdf/sensors/wamv_pinger.xacro" />
 </robot>

File: wamv_gazebo/urdf/sensors/wamv_camera.xacro (robot description, xacro)
@@ -38,8 +38,4 @@
           iyz="0"/>
       </inertial>
-    </link>
-    <!-- Define a link for the optical frame.  This will match the sensor frame and
-         be oriented in the camera convention. -->
-    <link name="${name}_link_optical">
     </link>
     <!-- Define post length and mass based on desired z position of sensor -->
@@ -120,11 +116,4 @@
       <child link="${name}_link" />
     </joint>
-    <!-- Camera to optical frame joint.  This is oriented to convert between ENU
-         and camera conventions -->
-    <joint name="${name}_to_${name}_link_optical_joint" type="fixed">
-      <origin xyz="0 0 0" rpy="${-pi/2} 0 ${-pi/2}" />
-      <parent link="${name}_link" />
-      <child link="${name}_link_optical" />
-    </joint>
     <!-- Gazebo camera setup -->
     <gazebo reference="${name}_link">
@@ -157,5 +146,5 @@
           <imageTopicName>image_raw</imageTopicName>
           <cameraInfoTopicName>camera_info</cameraInfoTopicName>
-          <frameName>${namespace}/${name}_link_optical</frameName>
+          <frameName>${name}_link_optical</frameName>
           <hackBaseline>0.07</hackBaseline>
           <distortionK1>0.0</distortionK1>

File: wamv_gazebo/urdf/sensors/wamv_gps.xacro (robot description, xacro)
@@ -25,7 +25,5 @@
       </inertial>
     </link>
-    <joint name="${name}_joint" type="revolute">
-      <axis xyz="0 0 1"/>
-      <limit effort="1000.0" lower="0.0" upper="0" velocity="0"/>
+    <joint name="${name}_joint" type="fixed">
       <origin xyz="${x} ${y} ${z}" rpy="${R} ${P} ${Y}" />
       <parent link="base_link" />
@@ -49,9 +47,9 @@
         <referenceLatitude>21.30996</referenceLatitude>
         <referenceLongitude>-157.8901</referenceLongitude>
-        <referenceAltitude>0</referenceAltitude>
+        <referenceAltitude>${z}</referenceAltitude>
         <referenceHeading>90</referenceHeading>
         <offset>0.0 0.0 0.0</offset>
         <drift>0.0 0.0 0.0</drift>
-        <gaussianNoise>0 0 0</gaussianNoise>
+        <gaussianNoise>0.1 0.1 0.1</gaussianNoise>
         <velocityOffset>0.0 0.0 0.0</velocityOffset>
         <velocityDrift>0.0 0.0 0.0</velocityDrift>

File: wamv_gazebo/urdf/sensors/wamv_imu.xacro (robot description, xacro)
@@ -11,12 +11,6 @@
         </material>
       </visual>
-      <inertial>
-        <mass value="0.1"/>
-        <inertia ixx="0.000083" ixy="0.0" ixz="0.0" iyy="0.000083" iyz="0.0" izz="0.0125"/>
-      </inertial>
     </link>
-    <joint name="${name}_joint" type="revolute">
-      <axis xyz="0 0 1"/>
-      <limit effort="1000.0" lower="0.0" upper="0" velocity="0"/>
+    <joint name="${name}_joint" type="fixed">
       <origin xyz="${x} ${y} ${z}" rpy="${R} ${P} ${Y}"/>
       <parent link="base_link"/>

File: wamv_gazebo/urdf/wamv_gazebo.urdf.xacro (robot description, xacro)
@@ -11,9 +11,7 @@
   <xacro:arg name="ground_truth_enabled" default="false" />
   <xacro:arg name="vrx_sensors_enabled" default="false" />
-  <xacro:arg name="pinger_enabled" default="false" />
   <xacro:arg name="thruster_namespace" default="thrusters/"/>
   <xacro:arg name="camera_namespace" default="cameras/"/>
   <xacro:arg name="sensor_namespace" default="sensors/"/>
-  <xacro:arg name="pinger_namespace" default="pingers/"/>
   <!-- Note: this is only used for some sensors that do not correctly use the
   robotNamespace parameter -->
@@ -22,5 +20,4 @@
   <xacro:property name="camera_namespace" value="$(arg camera_namespace)" scope="global" />
   <xacro:property name="sensor_namespace" value="$(arg sensor_namespace)" scope="global" />
-  <xacro:property name="pinger_namespace" value="$(arg pinger_namespace)" scope="global" />
   <xacro:property name="namespace" value="$(arg namespace)" scope="global" />
   <!-- Sensor yaml file -->
@@ -33,7 +30,12 @@
   <xacro:include filename="$(find wamv_gazebo)/urdf/wamv_gazebo.xacro"/>
   <!-- === Batteries === -->
+<!-->
   <xacro:include filename="$(find wamv_description)/urdf/battery.xacro"/>
   <xacro:battery prefix="left" position="0 1 0.45" orientation="0 0 0"/>
   <xacro:battery prefix="right" position="0 -1 0.45" orientation="0 0 0"/>
+<-->
+<!-- === RADAR === -->
+<xacro:include filename="$(find wamv_description)/urdf/radar.xacro"/>
+<xacro:radar prefix="main" position="-2.1 -0.1 2" orientation="0 0 0"/>
   <!-- === Thrusters === -->
   <!-- Use thruster yaml file if given -->
@@ -115,16 +117,15 @@
       <xacro:wamv_p3d name="p3d_wamv"/>
     </xacro:if>
-    <!-- Add pinger -->
-    <xacro:if value="$(arg pinger_enabled)">
-      <xacro:wamv_pinger name="pinger" position="1.0 0 -1.0" />
-    </xacro:if>
     <!-- ==== VRX sensor configuration ==== -->
     <xacro:if value="$(arg vrx_sensors_enabled)">
       <!-- Add CPU Cases -->
+<!-->
       <xacro:include filename="$(find wamv_description)/urdf/cpu_cases.xacro" />
       <xacro:cpu_cases position="-0.15 0 1.53" orientation="0 0 0"/>
+<-->
       <!-- Add a stereo camera pair -->
-      <xacro:wamv_camera name="front_left_camera" y="0.1" x="0.75" P="${radians(15)}" />
-      <xacro:wamv_camera name="front_right_camera" y="-0.1" x="0.75" P="${radians(15)}" />
+      <xacro:wamv_camera name="front_left_camera" y="0.5" x="0.75" z="0.75" post_Y="0.75" />
+      <xacro:wamv_camera name="front_right_camera" y="-0.5" x="0.75" z="0.75"  post_Y="0.75"/>
+<xacro:wamv_camera name="middle_camera" y="0" x="0.75" z="0.75"  post_Y="0.75"/>
       <!-- Add a camera facing right -->
       <xacro:wamv_camera name="middle_right_camera" y="-0.45" P="${radians(15)}" Y="${radians(-90)}" post_Y="${radians(-90)}" />
@@ -134,7 +135,5 @@
       <xacro:wamv_imu name="imu_wamv" y="-0.2" />
       <!-- Add 3D LIDAR -->
-      <xacro:lidar name="lidar_wamv" type="16_beam"/>
-      <!-- Add pinger -->
-      <xacro:wamv_pinger name="pinger" position="1.0 0 -1.0" />
+      <xacro:lidar name="lidar_wamv" x="1" y="0" z="1" type="16_beam"/>
     </xacro:if>
   </xacro:unless>
